File: STM32.kicad_sch (KiCad schematic)
At the start: 0 parts

Commit message: add full schematic
Parts:
- added C1, C2, C3, C4, C9: 100n, symbol Device:C
- added C10, C11: 10p, symbol Device:C
- added C12, C13: 22u, symbol Device:C
- added C5: 10u, symbol Device:C
- added C6: 10n, symbol Device:C
- added C7, C8: 1u, symbol Device:C
- added D1: RED, symbol Device:LED
- added FB1: 120R, symbol Device:FerriteBead
- added J1: USB_B_Micro, symbol Connector:USB_B_Micro
- added J2, J3, J4: Conn_01x04_Pin, symbol Connector:Conn_01x04_Pin
- added R1: 10k, symbol Device:R
- added R2, R3, R4, R5: 1.5k, symbol Device:R
- added SW1: SW_SPDT, symbol Switch:SW_SPDT
- added U1: STM32F103C8T6, Package_QFP:LQFP-48_7x7mm_P0.5mm, symbol MCU_ST_STM32F1:STM32F103C8Tx
- added U2: AMS1117-3.3, Package_TO_SOT_SMD:SOT-223-3_TabPin2, symbol Regulator_Linear:AMS1117-3.3
- added Y1: 16MHz, symbol Device:Crystal_GND24
Connections:
- new net +3.3V: C1.1, C13.1, C2.1, C3.1, C4.1, C5.1, C8.1, D1.2 (A), FB1.2, J2.1 (Pin_1), J3.1 (Pin_1), J4.1 (Pin_1), R2.1, R4.1, R5.1, SW1.3 (C), U1.1 (VBAT), U1.24 (VDD), U1.36 (VDD), U1.48 (VDD), U2.2 (VO)
- new net +3.3VA: C6.1, C7.1, FB1.1, U1.9 (VDDA)
- new net BOOT0: R1.2, U1.44 (BOOT0)
- new net GND: C1.2, C10.2, C11.2, C12.2, C13.2, C2.2, C3.2, C4.2, C5.2, C6.2, C7.2, C8.2, C9.2, J1.5 (GND), J2.4 (Pin_4), J3.4 (Pin_4), J4.4 (Pin_4), R3.2, SW1.1 (A), U1.23 (VSS), U1.35 (VSS), U1.47 (VSS), U1.8 (VSSA), U2.1 (GND), Y1.2 (G), Y1.4 (G)
- new net HSE_IN: C10.1, U1.5 (PD0), Y1.1
- new net HSE_OUT: C11.1, U1.6 (PD1), Y1.3
- new net I2C2_SCL: J4.2 (Pin_2), R4.2, U1.21 (PB10)
- new net I2C2_SDA: J4.3 (Pin_3), R5.2, U1.22 (PB11)
- new net NRST: C9.1, U1.7 (NRST)
- new net Power_Led_C: D1.1 (K), R3.1
- new net SWCLK: J2.3 (Pin_3), U1.37 (PA14)
- new net SWDIO: J2.2 (Pin_2), U1.34 (PA13)
- new net SW_BOOT0: R1.1, SW1.2 (B)
- new net USART1_RX: J3.3 (Pin_3), U1.43 (PB7)
- new net USART1_TX: J3.2 (Pin_2), U1.42 (PB6)
- new net USB_D+: J1.3 (D+), R2.2, U1.33 (PA12)
- new net USB_D-: J1.2 (D-), U1.32 (PA11)
- new net VBUS: C12.1, J1.1 (VBUS), U2.3 (VI)
- no-connect marks 0 -> 29
Other:
- note added: "CL=2*(CL0-Cs)=2*(10-5)pF=10pF"
- note added: "Microcontroller (and USB)"
- note added: "Phil's Lab PCB Learning Project - 1"
- note added: "Power Supply"
- note added: "USB App note AN4879"
- note added: "VBUS from USB Connector (nom. 5V) Min. 22uF inp/out capacitor"
- note added: "VDDA Filtering"
- title: (none) -> Phil's Lab Learning Project - 1

Commit message: add footprints
Parts:
- C1: renamed from C12; footprint (none) -> Capacitor_SMD:C_0805_2012Metric
- C10: renamed from C8; footprint (none) -> Capacitor_SMD:C_0402_1005Metric
- C11: renamed from C9; footprint (none) -> Capacitor_SMD:C_0402_1005Metric
- C12: renamed from C10; footprint (none) -> Capacitor_SMD:C_0402_1005Metric
- C13: renamed from C11; footprint (none) -> Capacitor_SMD:C_0402_1005Metric
- C2: renamed from C13; footprint (none) -> Capacitor_SMD:C_0805_2012Metric
- C3: renamed from C5; footprint (none) -> Capacitor_SMD:C_0603_1608Metric
- C4: footprint (none) -> Capacitor_SMD:C_0402_1005Metric
- C5: renamed from C3; footprint (none) -> Capacitor_SMD:C_0402_1005Metric
- C6: renamed from C2; footprint (none) -> Capacitor_SMD:C_0402_1005Metric
- C7: renamed from C1; footprint (none) -> Capacitor_SMD:C_0402_1005Metric
- C8: renamed from C6; footprint (none) -> Capacitor_SMD:C_0402_1005Metric
- C9: renamed from C7; footprint (none) -> Capacitor_SMD:C_0402_1005Metric
- D1: footprint (none) -> LED_SMD:LED_0603_1608Metric
- FB1: footprint (none) -> Inductor_SMD:L_0603_1608Metric
- J1: footprint (none) -> Connector_USB:USB_Micro-B_Wuerth_629105150521
- J2, J3, J4: footprint (none) -> Connector_PinHeader_2.54mm:PinHeader_1x04_P2.54mm_Vertical
- R1: renamed from R3; footprint (none) -> Resistor_SMD:R_0402_1005Metric
- R2: renamed from R1; footprint (none) -> Resistor_SMD:R_0402_1005Metric
- R3: renamed from R2; footprint (none) -> Resistor_SMD:R_0402_1005Metric
- R4, R5: footprint (none) -> Resistor_SMD:R_0402_1005Metric
- SW1: footprint (none) -> Button_Switch_THT:SW_E-Switch_EG1224_SPDT_Angled
- Y1: footprint (none) -> Crystal:Crystal_SMD_3225-4Pin_3.2x2.5mm
Changed lines of the file:
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@@
 			)
 		)
-		(property "Footprint" ""
+		(property "Footprint" "Connector_PinHeader_2.54mm:PinHeader_1x04_P2.54mm_Vertical"
 			(at 134.62 123.19 0)
 			(hide yes)
@@
 		(dnp no)
 		(fields_autoplaced yes)
-		(property "Reference" "C13"
+		(property "Reference" "C2"
 			(at 62.23 44.4499 0)
 			(show_name no)
@@
 			)
 		)
-		(property "Footprint" ""
+		(property "Footprint" "Capacitor_SMD:C_0805_2012Metric"
 			(at 59.3852 49.53 0)
 			(hide yes)
@@
 			(project "STM32"
 				(path "/96e5ad63-f918-4281-8426-104656eae99e"
-					(reference "C13")
+					(reference "C2")
 					(unit 1)
 				)
@@
 		(dnp no)
 		(fields_autoplaced yes)
-		(property "Reference" "C7"
+		(property "Reference" "C9"
 			(at 233.68 43.1799 0)
 			(show_name no)
@@
 			)
 		)
-		(property "Footprint" ""
+		(property "Footprint" "Capacitor_SMD:C_0402_1005Metric"
 			(at 230.8352 48.26 0)
 			(hide yes)
@@
 			(project "STM32"
 				(path "/96e5ad63-f918-4281-8426-104656eae99e"
-					(reference "C7")
+					(reference "C9")
 					(unit 1)
 				)
@@
 			)
 		)
-		(property "Footprint" ""
+		(property "Footprint" "Resistor_SMD:R_0402_1005Metric"
 			(at 154.178 140.97 90)
 			(hide yes)
@@
 		(dnp no)
 		(fields_autoplaced yes)
-		(property "Reference" "C1"
+		(property "Reference" "C7"
 			(at 189.23 44.4499 0)
 			(show_name no)
@@
 			)
 		)
-		(property "Footprint" ""
+		(property "Footprint" "Capacitor_SMD:C_0402_1005Metric"
 			(at 186.3852 49.53 0)
 			(hide yes)
@@
 			(project "STM32"
 				(path "/96e5ad63-f918-4281-8426-104656eae99e"
-					(reference "C1")
+					(reference "C7")
 					(unit 1)
 				)
@@
 			)
 		)
-		(property "Footprint" ""
+		(property "Footprint" "Button_Switch_THT:SW_E-Switch_EG1224_SPDT_Angled"
 			(at 157.48 64.77 0)
 			(hide yes)
@@
 			)
 		)
-		(property "Footprint" ""
+		(property "Footprint" "Connector_PinHeader_2.54mm:PinHeader_1x04_P2.54mm_Vertical"
 			(at 254 111.76 0)
 			(hide yes)
@@
 		(dnp no)
 		(fields_autoplaced yes)
-		(property "Reference" "C5"
+		(property "Reference" "C3"
 			(at 139.7 44.4499 0)
 			(show_name no)
@@
 			)
 		)
-		(property "Footprint" ""
+		(property "Footprint" "Capacitor_SMD:C_0603_1608Metric"
 			(at 136.8552 49.53 0)
 			(hide yes)
@@
 			(project "STM32"
 				(path "/96e5ad63-f918-4281-8426-104656eae99e"
-					(reference "C5")
+					(reference "C3")
 					(unit 1)
 				)
@@
 		(dnp no)
 		(fields_autoplaced yes)
-		(property "Reference" "C9"
+		(property "Reference" "C11"
 			(at 142.24 63.4999 0)
 			(show_name no)
@@
 			)
 		)
-		(property "Footprint" ""
+		(property "Footprint" "Capacitor_SMD:C_0402_1005Metric"
 			(at 139.3952 68.58 0)
 			(hide yes)
@@
 			(project "STM32"
 				(path "/96e5ad63-f918-4281-8426-104656eae99e"
-					(reference "C9")
+					(reference "C11")
 					(unit 1)
 				)
@@
 			)
 		)
-		(property "Footprint" ""
+		(property "Footprint" "Resistor_SMD:R_0402_1005Metric"
 			(at 156.972 140.97 90)
 			(hide yes)
@@
 		(dnp no)
 		(fields_autoplaced yes)
-		(property "Reference" "C8"
+		(property "Reference" "C10"
 			(at 251.46 43.1799 0)
 			(show_name no)
@@
 			)
 		)
-		(property "Footprint" ""
+		(property "Footprint" "Capacitor_SMD:C_0402_1005Metric"
 			(at 248.6152 48.26 0)
 			(hide yes)
@@
 			(project "STM32"
 				(path "/96e5ad63-f918-4281-8426-104656eae99e"
-					(reference "C8")
+					(reference "C10")
 					(unit 1)
 				)
@@
 			)
 		)
-		(property "Footprint" ""
+		(property "Footprint" "Capacitor_SMD:C_0402_1005Metric"
 			(at 149.5552 49.53 0)
 			(hide yes)
@@
 		(dnp no)
 		(fields_autoplaced yes)
-		(property "Reference" "C10"
+		(property "Reference" "C12"
 			(at 138.43 99.0599 0)
 			(show_name no)
@@
 			)
 		)
-		(property "Footprint" ""
+		(property "Footprint" "Capacitor_SMD:C_0402_1005Metric"
 			(at 135.5852 104.14 0)
 			(hide yes)
@@
 			(project "STM32"
 				(path "/96e5ad63-f918-4281-8426-104656eae99e"
-					(reference "C10")
+					(reference "C12")
 					(unit 1)
 				)
@@
 		(dnp no)
 		(fields_autoplaced yes)
-		(property "Reference" "C3"
+		(property "Reference" "C5"
 			(at 165.1 44.4499 0)
 			(show_name no)
@@
 			)
 		)
-		(property "Footprint" ""
+		(property "Footprint" "Capacitor_SMD:C_0402_1005Metric"
 			(at 162.2552 49.53 0)
 			(hide yes)
@@
 			(project "STM32"
 				(path "/96e5ad63-f918-4281-8426-104656eae99e"
-					(reference "C3")
+					(reference "C5")
 					(unit 1)
 				)
@@
 			)
 		)
-		(property "Footprint" ""
+		(property "Footprint" "Inductor_SMD:L_0603_1608Metric"
 			(at 240.03 41.148 90)
 			(hide yes)
@@
 		(dnp no)
 		(fields_autoplaced yes)
-		(property "Reference" "C6"
+		(property "Reference" "C8"
 			(at 220.98 43.1799 0)
 			(show_name no)
@@
 			)
 		)
-		(property "Footprint" ""
+		(property "Footprint" "Capacitor_SMD:C_0402_1005Metric"
 			(at 218.1352 48.26 0)
 			(hide yes)
@@
 			(project "STM32"
 				(path "/96e5ad63-f918-4281-8426-104656eae99e"
-					(reference "C6")
+					(reference "C8")
 					(unit 1)
 				)
@@
 		(dnp no)
 		(fields_autoplaced yes)
-		(property "Reference" "R2"
+		(property "Reference" "R3"
 			(at 242.57 81.2799 0)
 			(show_name no)
@@
 			)
 		)
-		(property "Footprint" ""
+		(property "Footprint" "Resistor_SMD:R_0402_1005Metric"
 			(at 238.252 82.55 90)
 			(hide yes)
@@
 			(project "STM32"
 				(path "/96e5ad63-f918-4281-8426-104656eae99e"
-					(reference "R2")
+					(reference "R3")
 					(unit 1)
 				)
@@
 		(dnp no)
 		(fields_autoplaced yes)
-		(property "Reference" "C12"
+		(property "Reference" "C1"
 			(at 34.29 44.4499 0)
 			(show_name no)
@@
 			)
 		)
-		(property "Footprint" ""
+		(property "Footprint" "Capacitor_SMD:C_0805_2012Metric"
 			(at 31.4452 49.53 0)
 			(hide yes)
@@
 			(project "STM32"
 				(path "/96e5ad63-f918-4281-8426-104656eae99e"
-					(reference "C12")
+					(reference "C1")
 					(unit 1)
 				)
@@
 			)
 		)
-		(property "Footprint" ""
+		(property "Footprint" "Connector_USB:USB_Micro-B_Wuerth_629105150521"
 			(at 257.81 86.36 0)
 			(hide yes)
@@
 			)
 		)
-		(property "Footprint" ""
+		(property "Footprint" "LED_SMD:LED_0603_1608Metric"
 			(at 67.31 39.37 0)
 			(hide yes)
@@
 			)
 		)
-		(property "Footprint" ""
+		(property "Footprint" "Crystal:Crystal_SMD_3225-4Pin_3.2x2.5mm"
 			(at 143.51 88.9 0)
 			(hide yes)
@@
 			)
 		)
-		(property "Footprint" ""
+		(property "Footprint" "Connector_PinHeader_2.54mm:PinHeader_1x04_P2.54mm_Vertical"
 			(at 134.62 146.05 0)
 			(hide yes)
@@
 		(dnp no)
 		(fields_autoplaced yes)
-		(property "Reference" "C11"
+		(property "Reference" "C13"
 			(at 157.48 99.0599 0)
 			(show_name no)
@@
 			)
 		)
-		(property "Footprint" ""
+		(property "Footprint" "Capacitor_SMD:C_0402_1005Metric"
 			(at 154.6352 104.14 0)
 			(hide yes)
@@
 			(project "STM32"
 				(path "/96e5ad63-f918-4281-8426-104656eae99e"
-					(reference "C11")
+					(reference "C13")
 					(unit 1)
 				)
@@
 		(dnp no)
 		(fields_autoplaced yes)
-		(property "Reference" "C2"
+		(property "Reference" "C6"
 			(at 177.8 44.4499 0)
 			(show_name no)
@@
 			)
 		)
-		(property "Footprint" ""
+		(property "Footprint" "Capacitor_SMD:C_0402_1005Metric"
 			(at 174.9552 49.53 0)
 			(hide yes)
@@
 			(project "STM32"
 				(path "/96e5ad63-f918-4281-8426-104656eae99e"
-					(reference "C2")
+					(reference "C6")
 					(unit 1)
 				)
@@
 		(dnp no)
 		(fields_autoplaced yes)
-		(property "Reference" "R3"
+		(property "Reference" "R1"
 			(at 81.28 44.4499 0)
 			(show_name no)
@@
 			)
 		)
-		(property "Footprint" ""
+		(property "Footprint" "Resistor_SMD:R_0402_1005Metric"
 			(at 76.962 45.72 90)
 			(hide yes)
@@
 			(project "STM32"
 				(path "/96e5ad63-f918-4281-8426-104656eae99e"
-					(reference "R3")
+					(reference "R1")
 					(unit 1)
 				)
@@
 		(in_pos_files yes)
 		(dnp no)
-		(property "Reference" "R1"
+		(property "Reference" "R2"
 			(at 171.704 60.706 90)
 			(show_name no)
@@
 			)
 		)
-		(property "Footprint" ""
+		(property "Footprint" "Resistor_SMD:R_0402_1005Metric"
 			(at 171.45 66.548 90)
 			(hide yes)
@@
 			(project "STM32"
 				(path "/96e5ad63-f918-4281-8426-104656eae99e"
-					(reference "R1")
+					(reference "R2")
 					(unit 1)
 				)

Commit message: layout components roughly in pcb
Parts:
- added H1, H2, H3, H4: MountingHole, MountingHole:MountingHole_2.2mm_M2, symbol Mechanical:MountingHole
- SW1: footprint Button_Switch_THT:SW_E-Switch_EG1224_SPDT_Angled -> Button_Switch_SMD:SW_SPDT_PCM12
Other:
- note added: "M2 Holes"
- note added: "Mounting Holes"

Commit message: route all components
Added a new footprint for the spdt switch as DRC was throwing a warning
Parts:
- SW1: footprint Button_Switch_SMD:SW_SPDT_PCM12 -> Boot_Switch:Boot_switch_custom
Changed lines of the file:
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@@
 			)
 		)
-		(property "Footprint" "Button_Switch_SMD:SW_SPDT_PCM12"
+		(property "Footprint" "Boot_Switch:Boot_switch_custom"
 			(at 157.48 64.77 0)
 			(hide yes)
